File: KiCad/RTC8088.kicad_pcb (KiCad board)
At the start: 2 copper layers, 86.4 x 38.1 mm, 11 parts, among them SW1 Address Select, U1 DS12885, U2 ATF16V8B, Y1 32768Hz

Commit message: Update silkscreen
Added logo aitorgomez.net
Other:
- board text added: "aitorgomez.net"
